File: elec/layout/default/sn65hvd230dr.kicad_pcb (KiCad board)
At the start: 2 copper layers, 225.7 x 100.8 mm, 0 parts

Commit message: layout
Parts:
- added C1: 16V 100nF X7R ±10% 0402 Multilayer Ceramic Capacitors MLCC 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, lib:C0402, F.Cu at (159.3, 107.0)
- added U1: , lib:SOIC-8_L4.9-W3.9-P1.27-LS6.0-BL, F.Cu at (159.4, 102.4)
Routing:
- net vcc: track 0.00 -> 1.93 mm
- net gnd: track 0.00 -> 1.91 mm
Changed lines of the file:
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@@
   )
   (net 0 "")
+  (net 1 "tx")
+  (net 2 "gnd")
+  (net 3 "vcc")
+  (net 4 "rx")
+  (net 5 "canh")
+  (net 6 "canl")
+  (net 7 "vref")
+  (footprint "lib:C0402" (layer "F.Cu")
+    (at 159.342691 106.996775 180)
+    (descr "Capacitor SMD 0402 (1005 Metric), square (rectangular) end terminal, IPC_7351 nominal, (Body size source: IPC-SM-782 page 76, https://www.pcb-3d.com/wordpress/wp-content/uploads/ipc-sm-782a_amendment_1_and_2.pdf), generated with kicad-footprint-generator")
+    (tags "capacitor")
+    (attr smd)
+    (fp_text reference "C1" (at 0 -1.16) (layer "F.SilkS")
+        (effects (font (size 1 1) (thickness 0.15)))
+    )
+    (fp_text value "16V 100nF X7R ±10% 0402  Multilayer Ceramic Capacitors MLCC - SMD/SMT ROHS" (at 0 1.16) (layer "F.Fab")
+        (effects (font (size 1 1) (thickness 0.15)))
+    )
+    (fp_text user "${REFERENCE}" (at 0 0) (layer "F.Fab")
+        (effects (font (size 0.25 0.25) (thickness 0.04)))
+    )
+    (fp_line (start -0.107836 -0.36) (end 0.107836 -0.36)
+      (stroke (width 0.12) (type solid)) (layer "F.SilkS"))
+    (fp_line (start -0.107836 0.36) (end 0.107836 0.36)
+      (stroke (width 0.12) (type solid)) (layer "F.SilkS"))
+    (fp_line (start -0.91 -0.46) (end 0.91 -0.46)
+      (stroke (width 0.05) (type solid)) (layer "F.CrtYd"))
+    (fp_line (start -0.91 0.46) (end -0.91 -0.46)
+      (stroke (width 0.05) (type solid)) (layer "F.CrtYd"))
+    (fp_line (start 0.91 -0.46) (end 0.91 0.46)
+      (stroke (width 0.05) (type solid)) (layer "F.CrtYd"))
+    (fp_line (start 0.91 0.46) (end -0.91 0.46)
+      (stroke (width 0.05) (type solid)) (layer "F.CrtYd"))
+    (fp_line (start -0.5 -0.25) (end 0.5 -0.25)
+      (stroke (width 0.1) (type solid)) (layer "F.Fab"))
+    (fp_line (start -0.5 0.25) (end -0.5 -0.25)
+      (stroke (width 0.1) (type solid)) (layer "F.Fab"))
+    (fp_line (start 0.5 -0.25) (end 0.5 0.25)
+      (stroke (width 0.1) (type solid)) (layer "F.Fab"))
+    (fp_line (start 0.5 0.25) (end -0.5 0.25)
+      (stroke (width 0.1) (type solid)) (layer "F.Fab"))
+    (pad "1" smd roundrect (at -0.48 0 180) (size 0.56 0.62) (layers "F.Cu" "F.Paste" "F.Mask") (roundrect_rratio 0.25)
+      (net 3 "vcc") (pintype "stereo"))
+    (pad "2" smd roundrect (at 0.48 0 180) (size 0.56 0.62) (layers "F.Cu" "F.Paste" "F.Mask") (roundrect_rratio 0.25)
+      (net 2 "gnd") (pintype "stereo"))
+    (model "${KICAD6_3DMODEL_DIR}/Capacitor_SMD.3dshapes/C_0402_1005Metric.wrl"
+      (offset (xyz 0 0 0))
+      (scale (xyz 1 1 1))
+      (rotate (xyz 0 0 0))
+    )
+  )
+  (footprint "lib:SOIC-8_L4.9-W3.9-P1.27-LS6.0-BL" (layer "F.Cu")
+    (at 159.355 102.37)
+    (attr smd)
+    (fp_text reference "U1" (at 0 -6.77) (layer "F.SilkS")
+        (effects (font (size 1 1) (thickness 0.15)))
+    )
+    (fp_text value "" (at 0 6.77) (layer "F.Fab")
+        (effects (font (size 1 1) (thickness 0.15)))
+    )
+    (fp_text user "${REFERENCE}" (at 0 0) (layer "F.Fab")
+        (effects (font (size 1 1) (thickness 0.15)))
+    )
+    (fp_line (start -2.53 -1.52) (end 2.53 -1.52)
+      (stroke (width 0.15) (type solid)) (layer "F.SilkS"))
+    (fp_line (start -2.53 1.52) (end -2.53 -1.52)
+      (stroke (width 0.15) (type solid)) (layer "F.SilkS"))
+    (fp_line (start 2.53 -1.52) (end 2.53 1.52)
+      (stroke (width 0.15) (type solid)) (layer "F.SilkS"))
+    (fp_line (start 2.53 1.52) (end -2.53 1.52)
+      (stroke (width 0.15) (type solid)) (layer "F.SilkS"))
+    (fp_circle (center -2.65 2.77) (end -2.5 2.77)
+      (stroke (width 0.3) (type solid)) (fill none) (layer "F.SilkS"))
+    (fp_circle (center -1.91 0.77) (end -1.76 0.77)
+      (stroke (width 0.3) (type solid)) (fill none) (layer "F.SilkS"))
+    (fp_circle (center -1.91 3.4) (end -1.76 3.4)
+      (stroke (width 0.3) (type solid)) (fill none) (layer "Cmts.User"))
+    (fp_circle (center -2.45 3) (end -2.42 3)
+      (stroke (width 0.06) (type solid)) (fill none) (layer "F.Fab"))
+    (pad "1" smd oval (at -1.91 2.77) (size 0.59 2.05) (layers "F.Cu" "F.Paste" "F.Mask")
+      (net 1 "tx") (pintype "stereo"))
+    (pad "2" smd oval (at -0.63 2.77) (size 0.59 2.05) (layers "F.Cu" "F.Paste" "F.Mask")
+      (net 2 "gnd") (pintype "stereo"))
+    (pad "3" smd oval (at 0.63 2.77) (size 0.59 2.05) (layers "F.Cu" "F.Paste" "F.Mask")
+      (net 3 "vcc") (pintype "stereo"))
+    (pad "4" smd oval (at 1.9 2.77) (size 0.59 2.05) (layers "F.Cu" "F.Paste" "F.Mask")
+      (net 4 "rx") (pintype "stereo"))
+    (pad "5" smd oval (at 1.9 -2.77) (size 0.59 2.05) (layers "F.Cu" "F.Paste" "F.Mask")
+      (net 7 "vref") (pintype "stereo"))
+    (pad "6" smd oval (at 0.63 -2.77) (size 0.59 2.05) (layers "F.Cu" "F.Paste" "F.Mask")
+      (net 6 "canl") (pintype "stereo"))
+    (pad "7" smd oval (at -0.63 -2.77) (size 0.59 2.05) (layers "F.Cu" "F.Paste" "F.Mask")
+      (net 5 "canh") (pintype "stereo"))
+    (pad "8" smd oval (at -1.91 -2.77) (size 0.59 2.05) (layers "F.Cu" "F.Paste" "F.Mask")
+      (net 2 "gnd") (pintype "stereo"))
+    (model "/Users/narayanpowderly/Documents/atopile-workspace/servo-drive/.ato/modules/sn65hvd230dr/elec/footprints/footprints.3dshapes/SOIC-8_L4.9-W3.9-H1.7-LS6.0-P1.27.wrl"
+      (offset (xyz 1.65 -2.84 -0))
+      (scale (xyz 1 1 1))
+      (rotate (xyz 0 0 0))
+    )
+  )
   (gr_circle (center 225.62 81.79) (end 227.32 81.79)
     (stroke (width 0.1) (type solid)) (fill none) (layer "Edge.Cuts"))
@@
       (xy 69.100734 49.778315)
     )
-    (stroke (width 0) (type solid)) (fill none) (layer "Edge.Cuts"))
+    (stroke (width 0.1) (type solid)) (fill none) (layer "Edge.Cuts"))
   (gr_arc (start 261.62 113.79) (mid 260.448427 116.618427) (end 257.62 117.79)
     (stroke (width 0.1) (type solid)) (layer "Edge.Cuts"))
@@
     (effects (font (size 2 2) (thickness 0.1)) (justify left bottom))
   )
+  (segment (start 158.725 106.859084) (end 158.862691 106.996775) (width 0.25) (layer "F.Cu") (net 2))
+  (segment (start 158.725 105.14) (end 158.725 106.859084) (width 0.25) (layer "F.Cu") (net 2))
+  (segment (start 159.991076 106.82839) (end 159.991076 105.146076) (width 0.25) (layer "F.Cu") (net 3))
+  (segment (start 159.991076 105.146076) (end 159.985 105.14) (width 0.25) (layer "F.Cu") (net 3))
+  (segment (start 159.822691 106.996775) (end 159.991076 106.82839) (width 0.25) (layer "F.Cu") (net 3))
   (group "" (id 6c1ef9f7-0f34-47bb-ac1a-76df23fb396e)
     (members
